Commit message: diff driv sim urdf tutorial

File: src/diff_drive_sim/resource/robot.urdf (robot description, URDF)
Before this commit: robot robot, 0 links, 0 joints
Links:
- added link base_link; collision box size=0.1 0.1 0.05; visual box size=0.1 0.1 0.05
- added link caster; collision sphere radius=0.0125; visual sphere radius=0.0125
- added link front_frame; collision cylinder length=0.05 radius=0.05; visual cylinder length=0.05 radius=0.05
- added link wheel1; collision cylinder length=0.02 radius=0.03; visual cylinder length=0.02 radius=0.03
- added link wheel2; collision cylinder length=0.02 radius=0.03; visual cylinder length=0.02 radius=0.03
Joints:
- added joint base_link_to_caster: type fixed, parent base_link, child caster, origin xyz=0 0.06 -0.0375 rpy=0 0 0
- added joint base_link_to_front_frame: type fixed, parent base_link, child front_frame, origin xyz=0 0.05 0 rpy=0 0 0
- added joint motor1: type continuous, parent base_link, child wheel1, origin xyz=0.06 0 -0.02 rpy=0 1.57 0, axis 0 0 1, limit effort=10 velocity=10
- added joint motor2: type continuous, parent base_link, child wheel2, origin xyz=-0.06 0 -0.02 rpy=0 1.57 0, axis 0 0 1, limit effort=10 velocity=10

Commit message: diff drive sim distance sensors

File: src/diff_drive_sim/resource/robot.urdf (robot description, URDF)
Before this commit: robot robot, 5 links, 4 joints
Links:
- removed link base_link
- removed link caster
- removed link front_frame
- removed link wheel1
- removed link wheel2
Joints:
- removed joint base_link_to_caster
- removed joint base_link_to_front_frame
- removed joint motor1
- removed joint motor2
