Commit message: diff drive sim robot reference frame correction

File: src/diff_drive_sim/resource/diff_drive.urdf (robot description, URDF)
Before this commit: robot robot, 5 links, 4 joints
Joints:
- joint base_link_to_caster: origin xyz=0 0.06 -0.0375 rpy=0 0 0 -> xyz=0.06 0 -0.0375 rpy=0 0 0
- joint base_link_to_front_frame: origin xyz=0 0.05 0 rpy=0 0 0 -> xyz=0.05 0 0 rpy=0 0 0
- joint motor1: origin xyz=0.06 0 -0.02 rpy=0 1.57 0 -> xyz=0 0.06 -0.02 rpy=1.57 0 0
- joint motor2: origin xyz=-0.06 0 -0.02 rpy=0 1.57 0 -> xyz=0 -0.06 -0.02 rpy=1.57 0 0

File: src/diff_drive_sim/resource/diff_drive_lidar.urdf (robot description, URDF)
Before this commit: robot robot, 6 links, 5 joints
Links:
- removed link lidar
Joints:
- removed joint base_link_to_lidar
- joint base_link_to_caster: origin xyz=0 0.06 -0.0375 rpy=0 0 0 -> xyz=0.06 0 -0.0375 rpy=0 0 0
- joint base_link_to_front_frame: origin xyz=0 0.05 0 rpy=0 0 0 -> xyz=0.05 0 0 rpy=0 0 0
- joint motor1: origin xyz=0.06 0 -0.02 rpy=0 1.57 0 -> xyz=0 0.06 -0.02 rpy=1.57 0 0
- joint motor2: origin xyz=-0.06 0 -0.02 rpy=0 1.57 0 -> xyz=0 -0.06 -0.02 rpy=1.57 0 0

Commit message: URDF updates

File: src/diff_drive_sim/resource/diff_drive.urdf (robot description, URDF)
Before this commit: robot robot, 5 links, 4 joints
Joints:
- joint motor1: axis 0 0 1 -> 0 0 -1
- joint motor2: axis 0 0 1 -> 0 0 -1

File: src/diff_drive_sim/resource/diff_drive_lidar.urdf (robot description, URDF)
Before this commit: robot robot, 5 links, 4 joints
Joints:
- joint motor1: axis 0 0 1 -> 0 0 -1
- joint motor2: axis 0 0 1 -> 0 0 -1
