Commit message: diff drive sim updates

File: src/diff_drive_sim/resource/diff_drive_lidar.urdf (robot description, URDF)
Before this commit: robot robot, 5 links, 4 joints
Links:
- added link lidar; collision cylinder length=0.025 radius=0.025; visual cylinder length=0.025 radius=0.025
Joints:
- added joint base_link_to_lidar: type fixed, parent base_link, child lidar, origin xyz=0 0 0.0375 rpy=0 0 0
