Commit message: Mecanum sim updates

File: src/mecanum_robot_sim/resource/robot.urdf (robot description, URDF)
Before this commit: robot robot, 7 links, 6 joints
Links:
- link base_link: geometry collision box size=0.3 0.2 0.1; visual box size=0.3 0.2 0.1
- link lidar: geometry collision cylinder length=0.05 radius=0.04; visual cylinder length=0.05 radius=0.04
- link wheel1: geometry collision cylinder length=0.04 radius=0.04; visual cylinder length=0.04 radius=0.04
- link wheel2: geometry collision cylinder length=0.04 radius=0.04; visual cylinder length=0.04 radius=0.04
- link wheel3: geometry collision cylinder length=0.04 radius=0.04; visual cylinder length=0.04 radius=0.04
- link wheel4: geometry collision cylinder length=0.04 radius=0.04; visual cylinder length=0.04 radius=0.04
Joints:
- joint base_link_lidar_joint: origin xyz=-0.04 0 0.096 rpy=0 0 0 -> xyz=0 0 0.075 rpy=0 0 0
- joint motor1: origin xyz=0.08 0 -0.055 rpy=1.57 0.000148 0 -> xyz=0.1 0.12 -0.035 rpy=1.57 0 0
- joint motor2: origin xyz=0.08 0 -0.055 rpy=1.57 -0.000151 0 -> xyz=0.1 -0.12 -0.035 rpy=1.57 0 0
- joint motor3: origin xyz=-0.08 0 -0.055 rpy=1.57 0.000157 0 -> xyz=-0.1 0.12 -0.035 rpy=1.57 0 0
- joint motor4: origin xyz=-0.08 0 -0.055 rpy=1.57 -0.000157 0 -> xyz=-0.1 -0.12 -0.035 rpy=1.57 0 0
