Commit message: Added rtabmap example

File: src/mecanum_robot_sim/resource/robot_camera.urdf (robot description, URDF)
Before this commit: robot robot, 8 links, 7 joints
Joints:
- joint base_link_to_camera: origin xyz=0.15 0 0 rpy=0 0 0 -> xyz=0.15 0 0 rpy=1.57 3.14 1.57

Commit message: rtabmap example updates

File: src/mecanum_robot_sim/resource/robot_camera.urdf (robot description, URDF)
Before this commit: robot robot, 8 links, 7 joints
Joints:
- joint base_link_to_camera: origin xyz=0.15 0 0 rpy=1.57 3.14 1.57 -> xyz=0.15 0 0 rpy=0 0 0
