Commit message: Updated launch files and added xacro description to mrs sim to correct frame names

File: src/rosmasterx3_sim/resource/rosmasterx3_multi_robot.urdf.xacro (robot description, xacro)
@@ -1,4 +1,7 @@
 <?xml version="1.0" encoding="utf-8"?>
-<robot name="robot">
+<robot xmlns:xacro="http://ros.org/wiki/xacro" name="robot">
+    <!-- declare the xacro arg/property immediately inside the robot root -->
+    <xacro:arg name="robot_name" default=""/>
+    <xacro:property name="robot_name" value="$(arg robot_name)"/>
     <!--#########-->
     <!-- PLUGINS -->
@@ -12,5 +15,5 @@
                 <topicName>scan</topicName>
                 <alwaysOn>true</alwaysOn>
-                <frameName>lidar</frameName>
+                <frameName>${robot_name}/lidar</frameName>
             </ros>
         </device>
@@ -20,5 +23,5 @@
             <updateRate>10</updateRate>
             <alwaysOn>True</alwaysOn>
-            <frameName>imu</frameName>
+            <frameName>${robot_name}/imu</frameName>
             <inertialUnitName>imu</inertialUnitName>
             <gyroName>gyro</gyroName>
@@ -31,5 +34,5 @@
                 <topicName>camera</topicName>
                 <alwaysOn>true</alwaysOn>
-                <frameName>optical_frame</frameName>
+                <frameName>${robot_name}/optical_frame</frameName>
             </ros>
         </device>
@@ -40,11 +43,11 @@
                 <topicName>range_finder</topicName>
                 <alwaysOn>true</alwaysOn>
-                <frameName>optical_frame</frameName>
+                <frameName>${robot_name}/optical_frame</frameName>
             </ros>
         </device>
     </webots>
-    <link name="base_footprint"/>
+    <link name="${robot_name}/base_footprint"/>
     <!-- Base Link -->
-    <link name="base_link">
+    <link name="${robot_name}/base_link">
         <inertial>
             <origin xyz="0.00498197982182523 5.70233829969297E-05 -0.0121008098068578" rpy="0 0 0"/>
@@ -74,18 +77,18 @@
         </collision>
     </link>
-    <joint name="base_joint" type="fixed">
-        <parent link="base_footprint"/>
-        <child link="base_link"/>
+    <joint name="${robot_name}/base_joint" type="fixed">
+        <parent link="${robot_name}/base_footprint"/>
+        <child link="${robot_name}/base_link"/>
         <origin xyz="0.0 0.0 0.0815" rpy="0 0 0"/>
     </joint>
     <!-- IMU -->
-    <link name="imu"/>
-    <joint name="base_imu" type="fixed">
-        <parent link="base_link"/>
-        <child link="imu"/>
+    <link name="${robot_name}/imu"/>
+    <joint name="${robot_name}/base_imu" type="fixed">
+        <parent link="${robot_name}/base_link"/>
+        <child link="${robot_name}/imu"/>
         <origin xyz="-0.06 0.01 0.01" rpy="0 3.1415 1.5707"/>
     </joint>
     <!-- Wheels -->
-    <link name="front_right_wheel">
+    <link name="${robot_name}/front_right_wheel">
         <inertial>
             <origin xyz="1.9051E-06 -2.3183E-07 -0.00064079" rpy="0 0 0"/>
@@ -110,12 +113,12 @@
         </collision>
     </link>
-    <joint name="front_right_joint" type="continuous">
+    <joint name="${robot_name}/front_right_joint" type="continuous">
         <origin xyz="0.08 -0.0845 -0.0389" rpy="-1.5703 0 3.14159"/>
-        <parent link="base_link"/>
-        <child link="front_right_wheel"/>
-        <axis xyz="0 0 1" rpy="0 0 0"/>
-        <limit effort="100" velocity="1"/>
-    </joint>
-    <link name="front_left_wheel">
+        <parent link="${robot_name}/base_link"/>
+        <child link="${robot_name}/front_right_wheel"/>
+        <axis xyz="0 0 1" rpy="0 0 0"/>
+        <limit effort="100" velocity="1"/>
+    </joint>
+    <link name="${robot_name}/front_left_wheel">
         <inertial>
             <origin xyz="2.3728E-06 -9.4228E-07 0.00064068" rpy="0 0 0"/>
@@ -140,12 +143,12 @@
         </collision>
     </link>
-    <joint name="front_left_joint" type="continuous">
+    <joint name="${robot_name}/front_left_joint" type="continuous">
         <origin xyz="0.08 0.084492 -0.0389" rpy="1.5703 0 0"/>
-        <parent link="base_link"/>
-        <child link="front_left_wheel"/>
-        <axis xyz="0 0 1" rpy="0 0 0"/>
-        <limit effort="100" velocity="1"/>
-    </joint>
-    <link name="back_right_wheel">
+        <parent link="${robot_name}/base_link"/>
+        <child link="${robot_name}/front_left_wheel"/>
+        <axis xyz="0 0 1" rpy="0 0 0"/>
+        <limit effort="100" velocity="1"/>
+    </joint>
+    <link name="${robot_name}/back_right_wheel">
         <inertial>
             <origin xyz="-1.75924169923403E-06 1.28388821071107E-06 -0.000590549296238266" rpy="0 0 0"/>
@@ -170,12 +173,12 @@
         </collision>
     </link>
-    <joint name="back_right_joint" type="continuous">
+    <joint name="${robot_name}/back_right_joint" type="continuous">
         <origin xyz="-0.08 -0.0845 -0.03946" rpy="-1.57 0 3.14159"/>
-        <parent link="base_link"/>
-        <child link="back_right_wheel"/>
-        <axis xyz="0 0 1" rpy="0 0 0"/>
-        <limit effort="100" velocity="1"/>
-    </joint>
-    <link name="back_left_wheel">
+        <parent link="${robot_name}/base_link"/>
+        <child link="${robot_name}/back_right_wheel"/>
+        <axis xyz="0 0 1" rpy="0 0 0"/>
+        <limit effort="100" velocity="1"/>
+    </joint>
+    <link name="${robot_name}/back_left_wheel">
         <inertial>
             <origin xyz="-4.01213085227115E-07 2.04910264598596E-06 0.000590775697051377" rpy="0 0 0"/>
@@ -200,12 +203,12 @@
         </collision>
     </link>
-    <joint name="back_left_joint" type="continuous">
+    <joint name="${robot_name}/back_left_joint" type="continuous">
         <origin xyz="-0.08 0.084492 -0.03954" rpy="1.5703 0 0"/>
-        <parent link="base_link"/>
-        <child link="back_left_wheel"/>
-        <axis xyz="0 0 1" rpy="0 0 0"/>
-        <limit effort="100" velocity="1"/>
-    </joint>
-    <link name="lidar">
+        <parent link="${robot_name}/base_link"/>
+        <child link="${robot_name}/back_left_wheel"/>
+        <axis xyz="0 0 1" rpy="0 0 0"/>
+        <limit effort="100" velocity="1"/>
+    </joint>
+    <link name="${robot_name}/lidar">
         <inertial>
             <origin xyz="-0.0176558922685589 0.000671805271544437 0.0219302095894866" rpy="0 0 0" />
@@ -230,10 +233,10 @@
         </collision>
     </link>
-    <joint name="lidar_joint" type="fixed">
+    <joint name="${robot_name}/lidar_joint" type="fixed">
         <origin xyz="0.0435 5.25826986680105E-05 0.11" rpy="0 0 0"/>
-        <parent link="base_link"/>
-        <child link="lidar"/>
-    </joint>
-    <link name="camera">
+        <parent link="${robot_name}/base_link"/>
+        <child link="${robot_name}/lidar"/>
+    </joint>
+    <link name="${robot_name}/camera">
         <inertial>
             <origin xyz="0 0 0" rpy="0 0 0"/>
@@ -257,8 +260,8 @@
         </collision>
     </link>
-    <joint name="camera_joint" type="fixed">
+    <joint name="${robot_name}/camera_joint" type="fixed">
         <origin xyz="0.057105 1.7948E-05 0.03755" rpy="0 0 0"/>
-        <parent link="base_link"/>
-        <child link="camera"/>
+        <parent link="${robot_name}/base_link"/>
+        <child link="${robot_name}/camera"/>
     </joint>
 </robot>
